Commit message: add upper spacers and lidar

File: urdf/design.urdf.xacro (robot description, xacro)
@@ -7,6 +7,11 @@
   <xacro:property name="wheel_radius" value="0.04"/>
   <xacro:property name="wheel_thickness" value="0.03"/>
+  <xacro:property name="spacer_radius" value="0.005"/>
+  <xacro:property name="spacer_thickness" value="0.1"/>
+  <xacro:property name="lidar_radius" value="0.06"/>
+  <xacro:property name="lidar_thickness" value="0.06"/>
 <!-- Main body -->
   <link name="world"/>
+  <!-- base -->
   <link name="base_link">
     <visual>
@@ -23,4 +28,20 @@
     <child link="base_link"/>
     <origin xyz="0 0 0.05" rpy="0 0 0"/>
+  </joint>
+  <!-- upper -->
+  <link name="upper_link">
+    <visual>
+      <geometry>
+        <box size="${body_length} ${body_width} ${body_height}"/>
+      </geometry>
+      <material name="red">
+        <color rgba="0.8 0 0 1"/>
+      </material>
+    </visual>
+  </link>
+  <joint name="base_to_upper" type="fixed">
+    <parent link="base_link"/>
+    <child link="upper_link"/>
+    <origin xyz="0 0 0.1" rpy="0 0 0"/>
   </joint>
   <!-- Wheel macro -->    <!-- macro is like a template -->
@@ -44,7 +65,45 @@
   </xacro:macro>
   <!-- Add four wheels -->
-  <xacro:wheel name="f_l"  x="0.09"  y="0.11" z="0.0"/>
-  <xacro:wheel name="f_r" x="0.09"  y="-0.11" z="0.0"/>
-  <xacro:wheel name="b_l"   x="-0.09" y="0.11" z="0.0"/>
-  <xacro:wheel name="b_r"  x="-0.09" y="-0.11" z="0.0"/>
+  <xacro:wheel name="fl_wheel"  x="0.09"  y="0.11"  z="0.0"/>
+  <xacro:wheel name="fr_wheel"  x="0.09"  y="-0.11" z="0.0"/>
+  <xacro:wheel name="bl_wheel"  x="-0.09" y="0.11"  z="0.0"/>
+  <xacro:wheel name="br_wheel"  x="-0.09" y="-0.11" z="0.0"/>
+  <!-- spacers macro -->
+  <xacro:macro name="spacer" params="name x y z">
+    <link name="${name}">
+      <visual>
+        <geometry>
+          <cylinder radius="${spacer_radius}" length="${spacer_thickness}"/>
+        </geometry>
+        <material name="yellow">
+          <color rgba="1 1 0 1"/>
+        </material>
+      </visual>
+    </link>
+    <joint name="${name}_joint" type="fixed">
+      <parent link="base_link"/>
+      <child link="${name}"/>
+      <origin xyz="${x} ${y} ${z}" rpy="0 0 0"/>
+    </joint>
+  </xacro:macro>
+  <!-- Add four spacers -->
+  <xacro:spacer name="fl_spacer" x="0.11"  y="0.08"  z="0.05"/>
+  <xacro:spacer name="fr_spacer" x="0.11"  y="-0.08" z="0.05"/>
+  <xacro:spacer name="bl_spacer" x="-0.11" y="0.08"  z="0.05"/>
+  <xacro:spacer name="br_spacer" x="-0.11" y="-0.08" z="0.05"/>
+  <link name="lidar_link">
+    <visual>
+      <geometry>
+        <cylinder radius="${lidar_radius}" length="${lidar_thickness}"/>
+      </geometry>
+      <material name="gary">
+        <color rgba="0.1 0.1 0.1 1"/>
+      </material>
+    </visual>
+  </link>
+  <joint name="lidar_to_upper" type="fixed">
+    <parent link="upper_link"/>
+    <child link="lidar_link"/>
+    <origin xyz="0.04 0 0.03" rpy="0 0.1 0"/>
+  </joint>
 </robot>

Commit message: launch gazebo

File: urdf/design.urdf.xacro (robot description, xacro)
@@ -23,4 +23,13 @@
       </material>
     </visual>
+    <collision>
+      <geometry>
+        <box size="${body_length} ${body_width} ${body_height}"/>
+      </geometry>
+    </collision>
+    <inertial>
+      <mass value="1.0"/>
+      <inertia ixx="0.01" iyy="0.01" izz="0.01" ixy="0" ixz="0" iyz="0"/>
+    </inertial>
   </link>
   <joint name="world_to_base" type="fixed">
@@ -39,4 +48,13 @@
       </material>
     </visual>
+    <collision>
+      <geometry>
+        <box size="${body_length} ${body_width} ${body_height}"/>
+      </geometry>
+    </collision>
+    <inertial>
+      <mass value="1.0"/>
+      <inertia ixx="0.01" iyy="0.01" izz="0.01" ixy="0" ixz="0" iyz="0"/>
+    </inertial>
   </link>
   <joint name="base_to_upper" type="fixed">
@@ -56,4 +74,13 @@
         </material>
       </visual>
+      <collision>
+        <geometry>
+          <cylinder radius="${wheel_radius}" length="${wheel_thickness}"/>
+        </geometry>
+      </collision>
+      <inertial>
+        <mass value="1.0"/> <!-- any values -->
+        <inertia ixx="0.01" iyy="0.01" izz="0.01" ixy="0" ixz="0" iyz="0"/>
+      </inertial>
     </link>
     <joint name="${name}_joint" type="continuous">
@@ -80,4 +107,13 @@
         </material>
       </visual>
+      <collision>
+        <geometry>
+          <cylinder radius="${spacer_radius}" length="${spacer_thickness}"/>
+        </geometry>
+      </collision>
+      <inertial>
+        <mass value="1.0"/> <!-- any values -->
+        <inertia ixx="0.01" iyy="0.01" izz="0.01" ixy="0" ixz="0" iyz="0"/>
+      </inertial>
     </link>
     <joint name="${name}_joint" type="fixed">
@@ -101,4 +137,13 @@
       </material>
     </visual>
+    <collision>
+      <geometry>
+        <cylinder radius="${lidar_radius}" length="${lidar_thickness}"/>
+      </geometry>
+    </collision>
+    <inertial>
+      <mass value="1.0"/>
+      <inertia ixx="0.01" iyy="0.01" izz="0.01" ixy="0" ixz="0" iyz="0"/>
+    </inertial>
   </link>
   <joint name="lidar_to_upper" type="fixed">

Commit message: fix wheel rotation

File: urdf/design.urdf.xacro (robot description, xacro)
@@ -88,5 +88,5 @@
       <child link="${name}"/>
       <origin xyz="${x} ${y} ${z}" rpy="1.57 0 0"/>
-      <axis xyz="0 1 0"/>
+      <axis xyz="0 0 1"/>
     </joint>
   </xacro:macro>

Commit message: fix inertial values

File: urdf/design.urdf.xacro (robot description, xacro)
@@ -29,6 +29,6 @@
     </collision>
     <inertial>
-      <mass value="1.0"/>
-      <inertia ixx="0.01" iyy="0.01" izz="0.01" ixy="0" ixz="0" iyz="0"/>
+      <mass value="0.5"/>
+      <inertia ixx="0.0017" iyy="0.00375" izz="0.0054" ixy="0" ixz="0" iyz="0"/>
     </inertial>
   </link>
@@ -54,6 +54,6 @@
     </collision>
     <inertial>
-      <mass value="1.0"/>
-      <inertia ixx="0.01" iyy="0.01" izz="0.01" ixy="0" ixz="0" iyz="0"/>
+      <mass value="0.5"/>
+      <inertia ixx="0.0017" iyy="0.00375" izz="0.0054" ixy="0" ixz="0" iyz="0"/>
     </inertial>
   </link>
@@ -80,6 +80,6 @@
       </collision>
       <inertial>
-        <mass value="1.0"/> <!-- any values -->
-        <inertia ixx="0.01" iyy="0.01" izz="0.01" ixy="0" ixz="0" iyz="0"/>
+        <mass value="0.025"/> <!-- any values -->
+        <inertia ixx="0.00002" iyy="0.00011" izz="0.00011" ixy="0" ixz="0" iyz="0"/>
       </inertial>
     </link>
@@ -113,6 +113,6 @@
       </collision>
       <inertial>
-        <mass value="1.0"/> <!-- any values -->
-        <inertia ixx="0.01" iyy="0.01" izz="0.01" ixy="0" ixz="0" iyz="0"/>
+        <mass value="0.0125"/> <!-- any values -->
+        <inertia ixx="0.000105" iyy="0.000105" izz="0" ixy="0" ixz="0" iyz="0"/>
       </inertial>
     </link>
@@ -143,6 +143,6 @@
     </collision>
     <inertial>
-      <mass value="1.0"/>
-      <inertia ixx="0.01" iyy="0.01" izz="0.01" ixy="0" ixz="0" iyz="0"/>
+      <mass value="0.05"/>
+      <inertia ixx="0.000225" iyy="0.000225" izz="0.00009" ixy="0" ixz="0" iyz="0"/>
     </inertial>
   </link>
@@ -150,5 +150,5 @@
     <parent link="upper_link"/>
     <child link="lidar_link"/>
-    <origin xyz="0.04 0 0.03" rpy="0 0.1 0"/>
+    <origin xyz="0.06 0 0.03" rpy="0 0.1 0"/>
   </joint>
 </robot>
